Commit message: Trying fully joint space planning with ompl

File: ur_moveit_config/srdf/ur_macro.srdf.xacro (robot description, xacro)
@@ -39,4 +39,12 @@
       <joint name="${prefix}wrist_3_joint" value="-0.11" />
     </group_state>
+    <group_state name="${prefix}test_configuration2" group="${prefix}${name}_manipulator">
+      <joint name="${prefix}elbow_joint" value="1.8" />
+      <joint name="${prefix}shoulder_lift_joint" value="-1.82" />
+      <joint name="${prefix}shoulder_pan_joint" value="-1.066" />
+      <joint name="${prefix}wrist_1_joint" value="-1.664" />
+      <joint name="${prefix}wrist_2_joint" value="-1.614" />
+      <joint name="${prefix}wrist_3_joint" value="-2.721" />
+    </group_state>
     <!--END EFFECTOR - Purpose - Represent information about an end effector.-->
     <!--VIRTUAL JOINT - Purpose - this element defines a virtual joint between a robot link and an external frame of reference (considered fixed with respect to the robot)-->
